File: PicoCIAA_Lora.kicad_pcb (KiCad board)
At the start: 2 copper layers, 51 x 30 mm, 8 parts, among them P3 PWR, P4 MOUNTING_HOLE, P5 MOUNTING_HOLE, P6 IO1, P8 IO3, U1 RFM95W, U2 EDGE_SMA

Commit message: PCB: ruteando
Parts:
- moved U1 12.5 mm to (70.5, 116.0)
- moved C2 2.10 mm to (69.0, 105.5)
Routing:
- net /DIO5: track 0.00 -> 38.4 mm
- net /nCS: track 0.00 -> 32.1 mm
- net /DIO3: track 0.00 -> 28.4 mm
- net /MOSI: track 0.00 -> 26.5 mm
- net /SCK: track 0.00 -> 26.2 mm
- net Net-(U1-Pad9): track 0.00 -> 25.5 mm
- net /DIO4: track 0.00 -> 23.1 mm
- net /MISO: track 0.00 -> 20.7 mm
Other:
- board size 51 x 30 mm -> 47 x 30 mm
- net class Default: clearance 0.2 -> 0
- rule trace_clearance: 0.2 -> 0
Changed lines of the file:
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@@
   (general
     (links 22)
-    (no_connects 22)
-    (area 48.999999 98.5904 112.433143 131.7358)
+    (no_connects 13)
+    (area 52.234286 98.5904 112.433143 131.7358)
     (thickness 1.6)
-    (drawings 19)
-    (tracks 0)
+    (drawings 8)
+    (tracks 50)
     (zones 0)
     (modules 8)
@@
   (setup
     (last_trace_width 0.25)
-    (trace_clearance 0.2)
+    (trace_clearance 0)
     (zone_clearance 0.508)
     (zone_45_only no)
@@
   (net 33 "Net-(P8-Pad10)")
   (net_class Default "This is the default net class."
-    (clearance 0.2)
+    (clearance 0)
     (trace_width 0.25)
     (via_dia 0.6)
@@
   )
   (module Capacitors_SMD:C_0402 (layer F.Cu)
-    (at 68.63 107.57 180)
+    (at 69 105.5 180)
     (descr "Capacitor SMD 0402, reflow soldering, AVX (see smccp.pdf)")
     (tags "capacitor 0402")
@@
       (effects (font (size 1 1) (thickness 0.15)))
     )
-    (fp_text value "0.1uF 10v" (at 0 1.27 180) (layer F.Fab)
+    (fp_text value "0.1uF 10v" (at 5.4 0.1 180) (layer F.Fab)
       (effects (font (size 1 1) (thickness 0.15)))
     )
@@
     (descr "Through hole pin header, 1x02, 2.00mm pitch, single row")
     (tags "pin header single row")
-    (fp_text reference P3 (at 0.775 -1.825 360) (layer F.SilkS)
-      (effects (font (size 1 1) (thickness 0.15)))
-    )
-    (fp_text value PWR (at 0 -3 270) (layer F.Fab)
+    (fp_text reference P3 (at -0.7 4.7 360) (layer F.SilkS)
+      (effects (font (size 1 1) (thickness 0.15)))
+    )
+    (fp_text value PWR (at 0.7 5.5 360) (layer F.Fab)
       (effects (font (size 1 1) (thickness 0.15)))
     )
@@
     (descr "Through hole pin header, 2x10, 2.00mm pitch, double row")
     (tags "pin header double row")
-    (fp_text reference P6 (at 3.7 17.4 360) (layer F.SilkS)
+    (fp_text reference P6 (at 4.275 7.075 360) (layer F.SilkS)
       (effects (font (size 1 1) (thickness 0.15)))
     )
@@
   )
   (module footprints:RFM95W (layer F.Cu)
-    (at 83 115.5)
+    (at 70.5 116)
     (fp_text reference U1 (at 0 3) (layer F.SilkS)
       (effects (font (size 1.5 1.5) (thickness 0.15)))
     )
-    (fp_text value RFM95W (at -13.53 1.09) (layer F.Fab)
-      (effects (font (size 1.5 1.5) (thickness 0.15)))
+    (fp_text value RFM95W (at -12.7 2) (layer F.Fab)
+      (effects (font (size 1.2 1.2) (thickness 0.15)))
     )
     (fp_line (start -8 -8) (end 8 -8) (layer F.SilkS) (width 0.15))
@@
     (descr "Through hole pin header, 2x05, 2.00mm pitch, double row")
     (tags "pin header double row")
-    (fp_text reference P8 (at 3.675 4.475 180) (layer F.SilkS)
-      (effects (font (size 1 1) (thickness 0.15)))
-    )
-    (fp_text value IO3 (at 0 -3 90) (layer F.Fab)
+    (fp_text reference P8 (at -0.5 10.875 180) (layer F.SilkS)
+      (effects (font (size 1 1) (thickness 0.15)))
+    )
+    (fp_text value IO3 (at 1.3 11.075 180) (layer F.Fab)
       (effects (font (size 1 1) (thickness 0.15)))
     )
@@
     )
   )
+  (gr_line (start 53 130) (end 100 130) (angle 90) (layer Edge.Cuts) (width 0.1))
+  (gr_line (start 53 100) (end 100 100) (angle 90) (layer Edge.Cuts) (width 0.1))
+  (gr_line (start 53 100) (end 53 130) (angle 90) (layer Edge.Cuts) (width 0.1))
   (gr_line (start 67.4 126) (end 67.4 129.5) (angle 90) (layer Edge.Cuts) (width 0.381))
   (gr_line (start 67.4 129.5) (end 73.4 129.5) (angle 90) (layer Edge.Cuts) (width 0.381))
   (gr_line (start 73.4 129.5) (end 73.4 126) (angle 90) (layer Edge.Cuts) (width 0.381))
   (gr_line (start 73.4 126) (end 67.4 126) (angle 90) (layer Edge.Cuts) (width 0.381))
-  (gr_arc (start 52.3 111.15) (end 53.05 111.15) (angle 90) (layer Edge.Cuts) (width 0.1))
-  (gr_line (start 100 130) (end 52.25 130) (angle 90) (layer Edge.Cuts) (width 0.1))
-  (gr_line (start 52.25 130) (end 52.25 128.65) (angle 90) (layer Edge.Cuts) (width 0.1))
-  (gr_arc (start 51.45 128.65) (end 51.45 127.85) (angle 90) (layer Edge.Cuts) (width 0.1))
-  (gr_line (start 51.45 127.85) (end 49.05 127.85) (angle 90) (layer Edge.Cuts) (width 0.1))
-  (gr_line (start 49.05 127.85) (end 49.05 111.9) (angle 90) (layer Edge.Cuts) (width 0.1))
-  (gr_line (start 49.05 111.9) (end 52.3 111.9) (angle 90) (layer Edge.Cuts) (width 0.1))
-  (gr_arc (start 52.3 111.15) (end 52.3 110.4) (angle 90) (layer Edge.Cuts) (width 0.1))
-  (gr_line (start 49.05 110.4) (end 52.3 110.4) (angle 90) (layer Edge.Cuts) (width 0.1))
-  (gr_line (start 49.05 102.15) (end 49.05 110.4) (angle 90) (layer Edge.Cuts) (width 0.1))
-  (gr_line (start 51.45 102.15) (end 49.05 102.15) (angle 90) (layer Edge.Cuts) (width 0.1))
-  (gr_arc (start 51.45 101.35) (end 52.25 101.35) (angle 90) (layer Edge.Cuts) (width 0.1))
-  (gr_line (start 52.25 100) (end 52.25 101.35) (angle 90) (layer Edge.Cuts) (width 0.1))
-  (gr_line (start 100 100) (end 52.25 100) (angle 90) (layer Edge.Cuts) (width 0.1))
   (gr_line (start 100 100) (end 100 130) (angle 90) (layer Edge.Cuts) (width 0.1))
+  (segment (start 89.675 101.725) (end 88.8 102.6) (width 0.25) (layer F.Cu) (net 4))
+  (segment (start 87.8 119) (end 77.5 119) (width 0.25) (layer F.Cu) (net 4))
+  (segment (start 88.8 118) (end 87.8 119) (width 0.25) (layer F.Cu) (net 4))
+  (segment (start 88.8 102.6) (end 88.8 118) (width 0.25) (layer F.Cu) (net 4))
+  (segment (start 87.675 101.725) (end 86.6 102.8) (width 0.25) (layer F.Cu) (net 5) (status 400000))
+  (segment (start 68.2 121) (end 63.5 121) (width 0.25) (layer F.Cu) (net 5) (status 800000))
+  (segment (start 75.2 114) (end 68.2 121) (width 0.25) (layer F.Cu) (net 5))
+  (segment (start 86 114) (end 75.2 114) (width 0.25) (layer F.Cu) (net 5))
+  (segment (start 86.6 113.4) (end 86 114) (width 0.25) (layer F.Cu) (net 5))
+  (segment (start 86.6 102.8) (end 86.6 113.4) (width 0.25) (layer F.Cu) (net 5))
+  (segment (start 81.675 101.725) (end 80.6 102.8) (width 0.25) (layer F.Cu) (net 8))
+  (segment (start 72.4 113) (end 63.5 113) (width 0.25) (layer F.Cu) (net 8))
+  (segment (start 72.8 112.6) (end 72.4 113) (width 0.25) (layer F.Cu) (net 8))
+  (segment (start 72.8 109.2) (end 72.8 112.6) (width 0.25) (layer F.Cu) (net 8))
+  (segment (start 75.4 106.6) (end 72.8 109.2) (width 0.25) (layer F.Cu) (net 8))
+  (segment (start 79.6 106.6) (end 75.4 106.6) (width 0.25) (layer F.Cu) (net 8))
+  (segment (start 80.6 105.6) (end 79.6 106.6) (width 0.25) (layer F.Cu) (net 8))
+  (segment (start 80.6 102.8) (end 80.6 105.6) (width 0.25) (layer F.Cu) (net 8))
+  (segment (start 63.5 117) (end 62 117) (width 0.25) (layer F.Cu) (net 10))
+  (segment (start 62 117) (end 60.4 115.4) (width 0.25) (layer F.Cu) (net 10))
+  (segment (start 60.4 115.4) (end 60.4 107.8) (width 0.25) (layer F.Cu) (net 10))
+  (segment (start 60.4 107.8) (end 61.6 106.6) (width 0.25) (layer F.Cu) (net 10))
+  (segment (start 61.6 106.6) (end 71.6 106.6) (width 0.25) (layer F.Cu) (net 10))
+  (segment (start 71.6 106.6) (end 73.2 105) (width 0.25) (layer F.Cu) (net 10))
+  (segment (start 73.2 105) (end 76 105) (width 0.25) (layer F.Cu) (net 10))
+  (segment (start 76 105) (end 76.6 104.4) (width 0.25) (layer F.Cu) (net 10))
+  (segment (start 76.6 104.4) (end 76.6 102.8) (width 0.25) (layer F.Cu) (net 10))
+  (segment (start 76.6 102.8) (end 77.675 101.725) (width 0.25) (layer F.Cu) (net 10))
+  (segment (start 87.675 103.725) (end 87.675 116.325) (width 0.25) (layer F.Cu) (net 15))
+  (segment (start 87 117) (end 77.5 117) (width 0.25) (layer F.Cu) (net 15))
+  (segment (start 87.675 116.325) (end 87 117) (width 0.25) (layer F.Cu) (net 15))
+  (segment (start 81.675 103.725) (end 81.675 105.725) (width 0.25) (layer F.Cu) (net 18))
+  (segment (start 72.4 115) (end 63.5 115) (width 0.25) (layer F.Cu) (net 18))
+  (segment (start 74 113.4) (end 72.4 115) (width 0.25) (layer F.Cu) (net 18))
+  (segment (start 74 109.6) (end 74 113.4) (width 0.25) (layer F.Cu) (net 18))
+  (segment (start 76 107.6) (end 74 109.6) (width 0.25) (layer F.Cu) (net 18))
+  (segment (start 79.8 107.6) (end 76 107.6) (width 0.25) (layer F.Cu) (net 18))
+  (segment (start 81.675 105.725) (end 79.8 107.6) (width 0.25) (layer F.Cu) (net 18))
+  (segment (start 79.675 103.725) (end 79.675 104.925) (width 0.25) (layer F.Cu) (net 19))
+  (segment (start 70.6 111) (end 63.5 111) (width 0.25) (layer F.Cu) (net 19))
+  (segment (start 71.2 110.4) (end 70.6 111) (width 0.25) (layer F.Cu) (net 19))
+  (segment (start 71.2 109) (end 71.2 110.4) (width 0.25) (layer F.Cu) (net 19))
+  (segment (start 74.4 105.8) (end 71.2 109) (width 0.25) (layer F.Cu) (net 19))
+  (segment (start 78.8 105.8) (end 74.4 105.8) (width 0.25) (layer F.Cu) (net 19))
+  (segment (start 79.675 104.925) (end 78.8 105.8) (width 0.25) (layer F.Cu) (net 19))
+  (segment (start 99.552 114.71) (end 97.266 114.71) (width 0.25) (layer F.Cu) (net 24) (status C00000))
+  (segment (start 97.266 114.71) (end 97.176 114.8) (width 0.25) (layer F.Cu) (net 24) (status C00000))
+  (segment (start 97.176 114.8) (end 94.2 114.8) (width 0.25) (layer F.Cu) (net 24) (status 400000))
+  (segment (start 94.2 114.8) (end 86 123) (width 0.25) (layer F.Cu) (net 24))
+  (segment (start 86 123) (end 77.5 123) (width 0.25) (layer F.Cu) (net 24) (status 800000))
 )

Commit message: PCB: completando ruteo
Parts:
- removed U2: EDGE_SMA, footprints:SMA_EDGE
- added P1: EDGE_SMA, footprints:SMA_EDGE, F.Cu at (106.2, 114.0)
- U1: value RFM95W -> RFM95
- moved C2 0.54 mm to (68.8, 105.0)
Routing:
- net /DIO0: track 0.00 -> 22.5 mm, vias 0 -> 1
- net /DIO1: track 0.00 -> 22.1 mm, vias 0 -> 1
- net +3V3: track 0.00 -> 18.2 mm, vias 0 -> 2
- net /DIO2: track 0.00 -> 16.9 mm, vias 0 -> 1
- net Net-(P1-Pad1): track 25.5 -> 27.3 mm
- added copper zone on B.Cu, net GND
- added copper zone on F.Cu, net GND
