File: PicoCIAA_Lora.sch (KiCad schematic (older format))
At the start: 8 parts, among them P3 PWR, P4 MOUNTING_HOLE, P5 MOUNTING_HOLE, P6 IO1, P8 IO3, U1 RFM95, U2 EDGE_SMA

Commit message: SCH: Actualizando esquema
Parts:
- removed U2: EDGE_SMA, footprints:SMA_EDGE, symbol EDGE_SMA
- added P1: EDGE_SMA, footprints:SMA_EDGE, symbol GSG-RF-CONN
Connections:
- net GND: now also P1.0, P1.2 (GND)
- net at U1.9 (ANT): now also P1.1 (RF)
Changed lines of the file:
@@
-$EndComp
-$Comp
-L EDGE_SMA U2
-U 1 1 592220FA
-P 5800 4050
-F 0 "U2" H 5850 3900 60  0000 C CNN
-F 1 "EDGE_SMA" H 5800 4250 60  0000 C CNN
-F 2 "footprints:SMA_EDGE" H 5800 4050 60  0001 C CNN
-F 3 "" H 5800 4050 60  0001 C CNN
-F 4 "Molex" H 5800 4050 60  0001 C CNN "Manf"
-F 5 "0732511150" H 5800 4050 60  0001 C CNN "Manf#"
-F 6 "WM5534-ND" H 5800 4050 60  0001 C CNN "Digikey#"
-F 7 "Value" H 5800 4050 60  0001 C CNN "Fieldname"
-	1    5800 4050
-	-1   0    0    1
 $EndComp
 $Comp
 L GND #PWR02
 U 1 1 5926212E
-P 6150 4400
-F 0 "#PWR02" H 6150 4150 50  0001 C CNN
-F 1 "GND" H 6150 4250 50  0000 C CNN
-F 2 "" H 6150 4400 50  0000 C CNN
-F 3 "" H 6150 4400 50  0000 C CNN
-	1    6150 4400
+P 6250 4400
+F 0 "#PWR02" H 6250 4150 50  0001 C CNN
+F 1 "GND" H 6250 4250 50  0000 C CNN
+F 2 "" H 6250 4400 50  0000 C CNN
+F 3 "" H 6250 4400 50  0000 C CNN
+	1    6250 4400
 	1    0    0    -1
 $EndComp
@@
 F 3 "" H 4900 3650 50  0000 C CNN
 	1    4900 3650
-	1    0    0    -1
-$EndComp
-$Comp
-L GND #PWR04
-U 1 1 5926263F
-P 5550 4400
-F 0 "#PWR04" H 5550 4150 50  0001 C CNN
-F 1 "GND" H 5550 4250 50  0000 C CNN
-F 2 "" H 5550 4400 50  0000 C CNN
-F 3 "" H 5550 4400 50  0000 C CNN
-	1    5550 4400
 	1    0    0    -1
 $EndComp
@@
 $EndComp
 $Comp
-L GND #PWR05
+L GND #PWR04
 U 1 1 592B4A0F
 P 7050 4100
-F 0 "#PWR05" H 7050 3850 50  0001 C CNN
+F 0 "#PWR04" H 7050 3850 50  0001 C CNN
 F 1 "GND" H 7050 3950 50  0000 C CNN
 F 2 "" H 7050 4100 50  0000 C CNN
@@
 $EndComp
 $Comp
-L GND #PWR06
+L GND #PWR05
 U 1 1 592B5BD6
 P 6200 3300
-F 0 "#PWR06" H 6200 3050 50  0001 C CNN
+F 0 "#PWR05" H 6200 3050 50  0001 C CNN
 F 1 "GND" H 6200 3150 50  0000 C CNN
 F 2 "" H 6200 3300 50  0000 C CNN
@@
 $EndComp
 $Comp
-L GND #PWR07
+L GND #PWR06
 U 1 1 592B5EA9
 P 4300 2650
-F 0 "#PWR07" H 4300 2400 50  0001 C CNN
+F 0 "#PWR06" H 4300 2400 50  0001 C CNN
 F 1 "GND" H 4300 2500 50  0000 C CNN
 F 2 "" H 4300 2650 50  0000 C CNN
@@
 Text Notes 2500 2200 0    60   ~ 0
 Uso del conector P6 de la PicoCIAA
-Wire Wire Line
-	5850 3250 5850 3800
-Wire Wire Line
-	6150 4000 6150 4400
-Wire Wire Line
-	4900 3250 4900 3650
-Wire Wire Line
-	5850 3150 6200 3150
-Connection ~ 6150 4100
-Wire Wire Line
-	5550 4000 5550 4400
-Connection ~ 5550 4100
-Wire Wire Line
-	4900 2750 4800 2750
-Wire Wire Line
-	4900 2850 4800 2850
-Wire Wire Line
-	4900 2650 4800 2650
-Wire Wire Line
-	4800 3150 4900 3150
-Wire Wire Line
-	5950 3050 5850 3050
-Wire Wire Line
-	5950 2950 5850 2950
-Wire Wire Line
-	5950 2750 5850 2750
-Wire Wire Line
-	5850 2550 5950 2550
-Wire Wire Line
-	5850 2650 5950 2650
-Wire Wire Line
-	3650 3100 3550 3100
-Wire Wire Line
-	2950 3100 3050 3100
-Wire Wire Line
-	3650 3200 3550 3200
-Wire Wire Line
-	3650 2600 3550 2600
-Wire Wire Line
-	3050 2600 2950 2600
-Wire Wire Line
-	3650 2700 3550 2700
-Wire Wire Line
-	3650 2800 3550 2800
-Wire Wire Line
-	3050 2700 2950 2700
-Wire Wire Line
-	7050 3750 7050 4100
-Wire Wire Line
-	7050 2600 7050 3450
-Wire Wire Line
-	4900 3050 4800 3050
-Wire Wire Line
-	6200 3150 6200 3300
-Connection ~ 7050 2850
-Wire Wire Line
-	4900 2550 4300 2550
-Wire Wire Line
-	4300 2550 4300 2650
-Wire Wire Line
-	3050 3300 2950 3300
-Wire Wire Line
-	4900 2950 4800 2950
-Wire Wire Line
-	3050 2800 2950 2800
-Wire Wire Line
-	5850 2850 7050 2850
-Wire Notes Line
-	2450 2050 4200 2050
-Wire Notes Line
-	4200 2050 4200 2250
-Wire Notes Line
-	4200 2250 2450 2250
-Wire Notes Line
-	2450 2250 2450 2050
 $Comp
 L CONN_01X01 P4
@@
 	1    0    0    -1
 $EndComp
-Wire Wire Line
-	8000 2500 8000 3100
-$Comp
-L GND #PWR08
+$Comp
+L GND #PWR07
 U 1 1 59452AC9
 P 8000 3100
-F 0 "#PWR08" H 8000 2850 50  0001 C CNN
+F 0 "#PWR07" H 8000 2850 50  0001 C CNN
 F 1 "GND" H 8000 2950 50  0000 C CNN
 F 2 "" H 8000 3100 50  0000 C CNN
@@
 	1    0    0    -1
 $EndComp
-Connection ~ 8000 2850
 $Comp
 L CONN_01X02 P3
@@
 $EndComp
 $Comp
-L +3.3V #PWR09
+L +3.3V #PWR08
 U 1 1 59454C80
 P 8600 3650
-F 0 "#PWR09" H 8600 3500 50  0001 C CNN
+F 0 "#PWR08" H 8600 3500 50  0001 C CNN
 F 1 "+3.3V" H 8600 3790 50  0000 C CNN
 F 2 "" H 8600 3650 50  0000 C CNN
@@
 $EndComp
 $Comp
-L GND #PWR010
+L GND #PWR09
 U 1 1 59454CA9
 P 8600 4150
-F 0 "#PWR010" H 8600 3900 50  0001 C CNN
+F 0 "#PWR09" H 8600 3900 50  0001 C CNN
 F 1 "GND" H 8600 4000 50  0000 C CNN
 F 2 "" H 8600 4150 50  0000 C CNN
@@
 	1    0    0    -1
 $EndComp
-Wire Wire Line
-	8600 3650 8600 3850
-Wire Wire Line
-	8600 3950 8600 4150
 $Comp
 L CONN_02X05 P8
@@
 NoConn ~ 3550 4400
 $Comp
-L GND #PWR011
+L GND #PWR010
 U 1 1 594DB5B8
 P 3050 4550
-F 0 "#PWR011" H 3050 4300 50  0001 C CNN
+F 0 "#PWR010" H 3050 4300 50  0001 C CNN
 F 1 "GND" H 3050 4400 50  0000 C CNN
 F 2 "" H 3050 4550 50  0000 C CNN
@@
 	1    0    0    -1
 $EndComp
-Wire Wire Line
-	3050 4400 3050 4550
-$Comp
-L PWR_FLAG #FLG?
+$Comp
+L PWR_FLAG #FLG011
 U 1 1 5960DE94
 P 8150 3700
-F 0 "#FLG?" H 8150 3795 50  0001 C CNN
+F 0 "#FLG011" H 8150 3795 50  0001 C CNN
 F 1 "PWR_FLAG" H 8150 3880 50  0000 C CNN
 F 2 "" H 8150 3700 50  0000 C CNN
@@
 $EndComp
 $Comp
-L PWR_FLAG #FLG?
+L PWR_FLAG #FLG012
 U 1 1 5960DEB8
 P 8150 4100
-F 0 "#FLG?" H 8150 4195 50  0001 C CNN
+F 0 "#FLG012" H 8150 4195 50  0001 C CNN
 F 1 "PWR_FLAG" H 8150 4280 50  0000 C CNN
 F 2 "" H 8150 4100 50  0000 C CNN
@@
 	1    0    0    -1
 $EndComp
+$Comp
+L GSG-RF-CONN P1
+U 1 1 596B9702
+P 5850 4150
+F 0 "P1" H 5850 4300 60  0000 C CNN
+F 1 "EDGE_SMA" V 5950 3800 60  0000 C CNN
+F 2 "footprints:SMA_EDGE" H 5850 4150 60  0001 C CNN
+F 3 "" H 5850 4150 60  0000 C CNN
+	1    5850 4150
+	0    -1   -1   0
+$EndComp
+Connection ~ 6250 4250
+Wire Wire Line
+	6250 4150 6250 4400
+Wire Wire Line
+	5850 3250 5850 3850
+Connection ~ 8600 4100
+Wire Wire Line
+	8150 4100 8600 4100
+Connection ~ 8600 3700
 Wire Wire Line
 	8150 3700 8600 3700
-Connection ~ 8600 3700
-Wire Wire Line
-	8150 4100 8600 4100
-Connection ~ 8600 4100
+Wire Wire Line
+	3050 4400 3050 4550
+Wire Wire Line
+	8600 3950 8600 4150
+Wire Wire Line
+	8600 3650 8600 3850
+Connection ~ 8000 2850
+Wire Wire Line
+	8000 2500 8000 3100
+Wire Notes Line
+	2450 2250 2450 2050
+Wire Notes Line
+	4200 2250 2450 2250
+Wire Notes Line
+	4200 2050 4200 2250
+Wire Notes Line
+	2450 2050 4200 2050
+Wire Wire Line
+	5850 2850 7050 2850
+Wire Wire Line
+	3050 2800 2950 2800
+Wire Wire Line
+	4900 2950 4800 2950
+Wire Wire Line
+	3050 3300 2950 3300
+Wire Wire Line
+	4300 2550 4300 2650
+Wire Wire Line
+	4900 2550 4300 2550
+Connection ~ 7050 2850
+Wire Wire Line
+	6200 3150 6200 3300
+Wire Wire Line
+	4900 3050 4800 3050
+Wire Wire Line
+	7050 2600 7050 3450
+Wire Wire Line
+	7050 3750 7050 4100
+Wire Wire Line
+	3050 2700 2950 2700
+Wire Wire Line
+	3650 2800 3550 2800
+Wire Wire Line
+	3650 2700 3550 2700
+Wire Wire Line
+	3050 2600 2950 2600
+Wire Wire Line
+	3650 2600 3550 2600
+Wire Wire Line
+	3650 3200 3550 3200
+Wire Wire Line
+	2950 3100 3050 3100
+Wire Wire Line
+	3650 3100 3550 3100
+Wire Wire Line
+	5850 2650 5950 2650
+Wire Wire Line
+	5850 2550 5950 2550
+Wire Wire Line
+	5950 2750 5850 2750
+Wire Wire Line
+	5950 2950 5850 2950
+Wire Wire Line
+	5950 3050 5850 3050
+Wire Wire Line
+	4800 3150 4900 3150
+Wire Wire Line
+	4900 2650 4800 2650
+Wire Wire Line
+	4900 2850 4800 2850
+Wire Wire Line
+	4900 2750 4800 2750
+Wire Wire Line
+	5850 3150 6200 3150
+Wire Wire Line
+	4900 3250 4900 3650
 $EndSCHEMATC

Commit message: PCB: Cambiando footprint capacitor a 0805
Parts:
- C2: footprint Capacitors_SMD:C_0402 -> Capacitors_SMD:C_0805
Changed lines of the file:
@@
 F 0 "C2" H 7075 3700 50  0000 L CNN
 F 1 "0.1uF 10v" H 7075 3500 50  0000 L CNN
-F 2 "Capacitors_SMD:C_0402" H 7088 3450 50  0001 C CNN
+F 2 "Capacitors_SMD:C_0805" H 7088 3450 50  0001 C CNN
 F 3 "" H 7050 3600 50  0000 C CNN
 F 4 "KEMET" H 7050 3600 60  0001 C CNN "Manf"
